File: uv_back/uv_back.kicad_sch (KiCad schematic)
At the start: 28 parts, among them J1 B3B-PH-SM4-TBT(LF)(SN), J2 B3B-PH-SM4-TBT(LF)(SN), J3 B3B-PH-SM4-TBT(LF)(SN), J4 B3B-PH-SM4-TBT(LF)(SN), J5 B3B-PH-SM4-TBT(LF)(SN)_ALT, J6 B3B-PH-SM4-TBT(LF)(SN)_ALT, J7 B3B-PH-SM4-TBT(LF)(SN), J8 B3B-PH-SM4-TBT(LF)(SN), J9 B3B-PH-SM4-TBT(LF)(SN)_ALT, SW1 CHS01TA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

Commit message: updated as built values
Parts:
- C1: DNP (none) -> 1
- C3: value 10000pF -> 0
- C4: value 1uF -> 4x 0.1uF
- R5, R7: value 1k -> 500
Changed lines of the file:
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@@
     (in_bom yes) (on_board yes)
     (property "Reference" "C4" (id 0) (at 275.59 177.8 90))
-    (property "Value" "1uF" (id 1) (at 275.59 185.42 90))
+    (property "Value" "4x 0.1uF" (id 1) (at 275.59 185.42 90))
     (property "Footprint" "Capacitor_SMD:C_0805_2012Metric_Pad1.18x1.45mm_HandSolder" (id 2) (at 279.4 180.6448 0)
       (effects (font (size 1.27 1.27)) hide)
@@
     (in_bom yes) (on_board yes)
     (property "Reference" "R5" (id 0) (at 181.61 154.94 90))
-    (property "Value" "1k" (id 1) (at 185.42 156.21 90))
+    (property "Value" "500" (id 1) (at 185.42 156.21 90))
     (property "Footprint" "Resistor_SMD:R_0805_2012Metric_Pad1.20x1.40mm_HandSolder" (id 2) (at 181.864 156.464 90)
       (effects (font (size 1.27 1.27)) hide)
@@
     (in_bom yes) (on_board yes)
     (property "Reference" "R7" (id 0) (at 180.34 195.58 90))
-    (property "Value" "1k" (id 1) (at 186.69 196.85 90))
+    (property "Value" "500" (id 1) (at 186.69 196.85 90))
     (property "Footprint" "Resistor_SMD:R_0805_2012Metric_Pad1.20x1.40mm_HandSolder" (id 2) (at 181.864 197.104 90)
       (effects (font (size 1.27 1.27)) hide)
@@
     (in_bom yes) (on_board yes)
     (property "Reference" "C3" (id 0) (at 247.65 139.7 90))
-    (property "Value" "10000pF" (id 1) (at 247.65 148.59 90))
+    (property "Value" "0" (id 1) (at 247.65 148.59 90))
     (property "Footprint" "Resistor_SMD:R_0805_2012Metric_Pad1.20x1.40mm_HandSolder" (id 2) (at 251.46 142.5448 0)
       (effects (font (size 1.27 1.27)) hide)
@@
       (effects (font (size 1.27 1.27)) hide)
     )
+    (property "DNP" "1" (id 4) (at 156.21 113.03 0)
+      (effects (font (size 1.27 1.27)) hide)
+    )
     (pin "1")
     (pin "2")
@@
     )
     (path "/b20f91e7-e5cb-49e4-bcc3-484b5358f6d1"
-      (reference "C3") (unit 1) (value "10000pF") (footprint "Resistor_SMD:R_0805_2012Metric_Pad1.20x1.40mm_HandSolder")
+      (reference "C3") (unit 1) (value "0") (footprint "Resistor_SMD:R_0805_2012Metric_Pad1.20x1.40mm_HandSolder")
     )
     (path "/05a0afb7-5c87-4d43-915d-28cebd0adf36"
-      (reference "C4") (unit 1) (value "1uF") (footprint "Capacitor_SMD:C_0805_2012Metric_Pad1.18x1.45mm_HandSolder")
+      (reference "C4") (unit 1) (value "4x 0.1uF") (footprint "Capacitor_SMD:C_0805_2012Metric_Pad1.18x1.45mm_HandSolder")
     )
     (path "/951ec362-b3ed-49fd-935b-718ed65c2d2d"
@@
     )
     (path "/3d3b8846-d3f5-4798-8bde-8f3581fdcc01"
-      (reference "R5") (unit 1) (value "1k") (footprint "Resistor_SMD:R_0805_2012Metric_Pad1.20x1.40mm_HandSolder")
+      (reference "R5") (unit 1) (value "500") (footprint "Resistor_SMD:R_0805_2012Metric_Pad1.20x1.40mm_HandSolder")
     )
     (path "/e940c989-d5b1-4a34-84a5-dd381089618c"
@@
     )
     (path "/9e13efff-464f-4a52-9c57-4be330a8375d"
-      (reference "R7") (unit 1) (value "1k") (footprint "Resistor_SMD:R_0805_2012Metric_Pad1.20x1.40mm_HandSolder")
+      (reference "R7") (unit 1) (value "500") (footprint "Resistor_SMD:R_0805_2012Metric_Pad1.20x1.40mm_HandSolder")
     )
     (path "/e9b4e634-30c2-46ef-9661-a2511ffb8282"
